File: DV-INT/VCU/VCU_itr2.brd (EAGLE design)
At the start: 160 x 100 mm, 67 parts, among them IC1 UCC2946D, IC11 74HC238D, IC12 LM324D, IC2 4081N, IC3 4071N, IC4 4081N, IC5 SI4425FDY-T1-GE3, IC6 L7805CV-DG, IC7 SI4425FDY-T1-GE3, IC8 4081N

Commit message: VCU Schematic Updated
Parts:
- removed IC11: 74HC238D, 74HC238D:SOIC127P600X175-16N
- removed IC12: LM324D, linear:SO14
- removed U$10, U$4, U$5, U$6, U$7, U$8: TSOP-6_NMOS, ACU-MOSFET-updated:TSOP-6_NMOS
- added C1, C12, C9: 100nF/0.1uF, IIT_BOMBAY_Racing:C0805
- added C10: 1uF, IIT_BOMBAY_Racing:SMC_A
- added C11: 2uF, IIT_BOMBAY_Racing:E2,5-6
- added C8: 10nF/0.01uF, IIT_BOMBAY_Racing:C0805
- added FB_POT: 17k, IIT_BOMBAY_Racing:S63S
- added FUSE_1A2: 1206L, IIT_BOMBAY_Racing2:1206L
- added IC9: 74HC238D, 74HC238D:SOIC127P600X175-16N
- added K1: CPC1002NSOP, CPC1002N:SOP04
- added LED->1, LED->2, LED->3, LED->4, LED->5, LED->6, LED->95: (no value), IIT_BOMBAY_Racing:FKIT-LED-1206
- added R16: 33k, IIT_BOMBAY_Racing2:M0805
- added R17, R19, R24, R26, R28, R42, R44: 100k, IIT_BOMBAY_Racing:R0805
- added R18, R22, R25, R27, R35, R43, R45: 10k, IIT_BOMBAY_Racing2:M0805
- added SI5, SI6, SI7: TSOP-6_PMOS, TSOP-6_MOS:TSOP-6_PMOS
- added U$13, U$16, U$17, U$18, U$19: TSOP-6_NMOS, ACU-MOSFET-updated:TSOP-6_NMOS
- added U1: LM324, LM324:SOIC127P600X175-14N
- added U2: SN74HC193QPWRG4Q1, counter_3bit:PW16
- IC2: value 4081N -> LM555N; device 40xx:DIL14 -> linear:DIL08
- IC3: value 4071N -> 4081N; device 40xx:DIL14 -> IIT_BOMBAY_Racing:DIL14
- IC4: device 40xx:DIL14 -> IIT_BOMBAY_Racing:DIL14
- IC8: value 4081N -> 4071N
- R1: value 51k -> 30k
- R10, R6: value 10k -> 5k; device IIT_BOMBAY_Racing2:M0805 -> IIT_BOMBAY_Racing:R0805
- R11, R12: value 100k -> 5k
- R13: value 10k -> 5k
- R14: value 100k -> 20k; device IIT_BOMBAY_Racing2:M0805 -> IIT_BOMBAY_Racing:R0805
- R15: device IIT_BOMBAY_Racing2:M0805 -> IIT_BOMBAY_Racing:R0805
- R2: value 10k -> 20k
- R20, R23, R29, R36, R40: device IIT_BOMBAY_Racing:R0805 -> IIT_BOMBAY_Racing2:M0805
- R31: value 100k -> 10k
- R32: value 10k -> 100k
- R33, R38: value 100k -> 10k; device IIT_BOMBAY_Racing:R0805 -> IIT_BOMBAY_Racing2:M0805
- R5, R7: value 100k -> 5k; device IIT_BOMBAY_Racing2:M0805 -> IIT_BOMBAY_Racing:R0805
- U$3: value TSOP-6_NMOS -> TEENSY40; device ACU-MOSFET-updated:TSOP-6_NMOS -> teensy:TEENSY40
- moved R23 276.0 mm to (-87.6, -209.6)
- moved IC8 221.5 mm to (-78.7, -200.7)
- moved D2 216.2 mm to (-86.4, -168.9)
- moved IC4 212.5 mm to (-78.7, -189.2)
- moved U$2 210.9 mm to (-88.9, -163.8)
- moved IC3 205.8 mm to (-78.7, -177.8)
- moved C3 201.4 mm to (-87.6, -154.9)
- moved SI4 137.8 mm to (-88.9, -81.3)
- moved R7 109.9 mm to (-77.5, -30.5)
- moved R6 108.5 mm to (-82.5, -30.5)
- moved U$3 106.0 mm to (-71.1, -62.2)
- moved R12 98.8 mm to (-82.5, -24.1)
- moved R13 98.5 mm to (-77.5, -24.1)
- moved R10 98.5 mm to (-87.6, -24.1)
- moved R11 96.6 mm to (-72.4, -24.1)
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- renumbered U$11 to U$14, U$12 to U$15
Connections:
- net +3V3 renamed +3V3_REF
- removed net +12V_AS: C2.2, D1.C, U$9.NO+, U$9.V+, X2.P$9
- removed net 2V_REF: R1.1, R2.2, U$1.2, U$1.5
- removed net 3V3: IC11.16, IC11.6
- removed net ASMS_STATE: IC2.2, IC4.6, R5.2, SI2.G, U$9.NO-, X2.P$10
- removed net IN1: IC11.1, IC12.1, IC12.2
- removed net IN1_IN: IC12.3
- removed net IN2: IC11.2, IC12.6, IC12.7
- removed net IN2_IN: IC12.5
- removed net IN3: IC11.3, IC12.8, IC12.9
- removed net IN3_IN: IC12.10
- removed net WATCHDOG_OUT: IC1.5, R11.2, U$3.G
- removed net WATCHDOG_OUT_12V: IC2.1, R23.1, U$3.1, U$3.2, U$3.5, U$3.6, U$3.D
- new net +12V_ASMS: C11.+, C2.2, D1.C, IC3.2, IC4.12, IC5.1, IC5.2, IC5.3, IC7.1, IC7.2, IC7.3, R20.2, R8.1, R9.1, SI4.S, SI5.G, U$1.8, U$9.V+
- new net 2VREF: R1.1, R2.2, U$1.2, U$1.5, U1.13, U1.2, U1.6, U1.9
- new net 3V3REF: FB_POT.E, IC9.16, IC9.6, R16.2
- new net AMI_0: IC9.1, U2.3
- new net AMI_1: IC9.2, U2.2
- new net AMI_2: IC9.3, U2.6
- new net ASMS_IN: U$9.NO+, X2.P$9
- new net ASMS_SUPPLY: C10.+, FUSE_1A2.P$1, U$9.NO-, X2.P$10
- new net AS_LATCH: IC2.3, R32.2, SI2.G
- new net AS_LATCH_INV: R33.2, R34.2, SI2.1, SI2.2, SI2.5, SI2.6, SI2.D
- new net AS_RELAY: R40.2, SI3.G, U1.14
- new net AS_RELAY_INV: C3.2, D2.C, R41.2, SI3.1, SI3.2, SI3.5, SI3.6, SI3.D, U$2.P$1
- new net AS_TRIG: IC2.2, IC8.11
- new net EBS_RESET: X2.P$7
- new net INIT_CHK_INV: IC8.5, U1.3
- new net INIT_CHK_INV_12V: IC8.13, K1.4, U1.1
- new net K2_RES: BMS-CONN7.P$6
- new net K3_RES: BMS-CONN7.P$5
- new net N$10: IC3.3, IC3.8
- new net N$11: IC3.4, IC3.9
- new net N$12: IC3.11, IC4.1
- new net N$13: LED->5.A, R12.2
- new net N$14: LED->6.A, R13.2
- new net N$15: K1.1, R14.1
- new net N$16: R34.1, R38.1, R39.1, U1.12
- new net N$18: C1.1, IC2.5
- new net N$19: C9.1, IC2.6, IC2.7
- new net N$20: R23.1, U2.14, U2.7
- new net N$21: U2.5
- new net N$28: LED->95.A, R5.2
- new net N$7: FUSE_1A2.P$2, SI4.1, SI4.2, SI4.5, SI4.6, SI4.D
- new net SIG5: IC4.13, IC8.4
- new net SIG6: K1.3, R15.1, R38.2
- new net WD_OUT: IC1.5, U1.5
- new net WD_OUT_12V: IC3.1, U1.7
- net +12V: now also C8.1, IC2.8, R20.1, R29.1, R31.2, R32.1, R36.1, R40.1, SI5.S, SI6.S, SI7.S, U$13.1, U$13.2, U$13.5, U$13.6, U$13.D, U$16.1, U$16.2, U$16.5, U$16.6, U$16.D, U$17.1, U$17.2, U$17.5, U$17.6, U$17.D, U$18.1, U$18.2, U$18.5, U$18.6, U$18.D, U$19.1, U$19.2, U$19.5, U$19.6, U$19.D, U1.4; no longer IC2.14, IC5.1, IC5.2, IC5.3, IC7.1, IC7.2, IC7.3, R1.2, R13.2, R14.1, R23.2, R5.1, R7.1, R8.1, R9.1, SI4.S, U$1.8, U$10.1, U$10.2, U$10.5, U$10.6, U$10.D, U$5.1, U$5.2, U$5.5, U$5.6, U$5.D, U$6.1, U$6.2, U$6.5, U$6.6, U$6.D, U$7.1, U$7.2, U$7.5, U$7.6, U$7.D, U$8.1, U$8.2, U$8.5, U$8.6, U$8.D
- net +5V: now also FB_POT.A, FB_POT.S, R1.2, U2.11, U2.16, U2.4
- net ACCELERATION: now also R13.1, R17.1, R18.2, U$13.S; no longer R20.1, R21.2, U$5.S
- net ACCELERATION_IN: now also IC9.15, R17.2, U$13.G; no longer IC11.15, R20.2, U$5.G
- net ASMS_STATE_INV: now also IC3.12, R21.2, SI5.1, SI5.2, SI5.5, SI5.6, SI5.D; no longer IC4.2, R6.2, SI2.1, SI2.2, SI2.5, SI2.6, SI2.D
- net AS_LOGIC: now also IC4.4, IC8.12, R14.2; no longer C3.2, D2.C, IC3.3, U$2.P$1
- net AUTOCROSS: now also R42.1, R43.2, R5.1, U$18.S; no longer R38.1, R39.2, U$14.S
- net AUTOCROSS_IN: now also IC9.13, R42.2, U$18.G; no longer IC11.13, R38.2, U$14.G
- net EBS_TEST: now also R24.1, R25.2, R7.1, U$15.S; no longer R31.1, R32.2, U$7.S, X2.P$7
- net EBS_TEST_IN: now also IC9.11, R24.2, U$15.G; no longer IC11.11, R31.2, U$7.G
- net GND: now also C1.2, C10.-, C11.-, C12.2, C8.2, C9.2, IC2.1, IC9.4, IC9.5, IC9.8, K1.2, LED->1.C, LED->2.C, LED->3.C, LED->4.C, LED->5.C, LED->6.C, LED->95.C, R15.2, R16.1, R18.1, R22.1, R23.2, R25.1, R27.1, R33.1, R35.1, R39.2, R43.1, R45.1, SI4.G, U1.11, U2.1, U2.10, U2.15, U2.8, U2.9; no longer IC11.4, IC11.5, IC11.8, IC12.11, IC2.7, R10.1, R11.1, R12.1, R15.1, R32.1, R34.1, R39.1, R6.1, U$3.S, U$4.S
- net HV_RESET: now also IC8.3; no longer IC3.4
- net HV_RESET_CP: now also IC4.9; no longer IC4.1
- net HV_RESET_SP: now also IC8.6; no longer IC4.5
- net INSPECTION: now also R10.1, R26.1, R27.2, U$16.S; no longer R33.1, R34.2, U$8.S
- net INSPECTION_IN: now also IC9.10, R26.2, U$16.G; no longer IC11.10, R33.2, U$8.G
- net MANUAL_DRIVING: now also IC3.13, R11.1, R29.2, R44.1, R45.2, SI6.G, U$19.S; no longer IC4.9, R40.1, R41.2, R7.2, SI3.G, U$15.S
- net MANUAL_DRIVING_IN: now also IC9.9, R44.2, U$19.G; no longer IC11.9, R40.2, U$15.G
- net MANUAL_DRIVING_INV: now also IC3.5, R30.2, SI6.1, SI6.2, SI6.5, SI6.6, SI6.D; no longer IC2.12, R10.2, SI3.1, SI3.2, SI3.5, SI3.6, SI3.D
- net MANUAL_VALVE: now also IC3.6, R36.2, SI7.G; no longer IC2.6, R14.2, SI4.G
- net MANUAL_VALVE_INV: now also IC4.2, R37.2, SI7.1, SI7.2, SI7.5, SI7.6, SI7.D; no longer IC4.12, R15.2, SI4.1, SI4.2, SI4.5, SI4.6, SI4.D
- net MISSION_SET: now also U1.10; no longer IC4.13, R12.2, U$4.G
- net MISSION_SET_12V: now also IC4.6, U1.8; no longer IC2.5, R13.1, U$4.1, U$4.2, U$4.5, U$4.6, U$4.D
- net N$17: now also C12.1, IC2.4, R31.1; no longer IC12.4
- net N$2: now also IC4.5, IC8.10; no longer IC2.3, IC2.8
- net N$4: now also LED->2.A, R7.2; no longer IC4.10, IC8.1
- net N$5: now also LED->4.A, R11.2; no longer IC2.4, IC2.9
- net N$6: now also LED->1.A, R6.2; no longer IC4.11, IC8.2
- net N$8: now also LED->3.A, R10.2; no longer IC2.11, IC3.1
- net SIG1: now also IC3.10, IC8.8; no longer IC2.10, IC2.13
- net SIG2: now also IC4.10, IC8.1; no longer IC3.5, IC4.3
- net SIG3: now also IC4.11, IC8.2; no longer IC3.6, IC4.4
- net SIG4: now also IC4.3, IC8.9; no longer IC3.2, IC8.3
- net SKIDPAD: now also R12.1, R19.1, R22.2, U$14.S; no longer R29.1, R30.2, U$6.S
- net SKIDPAD_IN: now also IC9.14, R19.2, U$14.G; no longer IC11.14, R29.2, U$6.G
- net TRACKDRIVE: now also R28.1, R35.2, R6.1, U$17.S; no longer R36.1, R37.2, U$10.S, X2.P$6
- net TRACKDRIVE_IN: now also IC9.12, R28.2, U$17.G; no longer IC11.12, R36.2, U$10.G
