File: DV-INT/VCU/VCU_itr2.sch (EAGLE design)
At the start: 95 parts, among them IC1 UCC2946D, IC10 LM324D, IC11 4081N, IC12 4071N, IC13 4081N, IC2 LM555N, IC5 SI4425FDY-T1-GE3, IC6 L7805CV-DG, IC7 SI4425FDY-T1-GE3, IC9 74HC238D, K1 CPC1002NSOP, U1 LM324

Commit message: VCU Schematic Updated
Parts:
- removed IC10: LM324D, linear:LM324D
- removed IC11, IC13: 4081N, 40xx:4081N
- removed IC12: 4071N, 40xx:4071N
- added C10: 1uF, IIT_BOMBAY_Racing:CPOL-EUSMCA
- added C11: 2uF, IIT_BOMBAY_Racing:CPOL-EUE2.5-6
- added C12: 100nF/0.1uF, IIT_BOMBAY_Racing:C-EUC0805
- added FUSE_1A2: 1206L, IIT_BOMBAY_Racing2:1206L
- added IC3, IC4: 4081N, IIT_BOMBAY_Racing:4081N
- added IC8: 4071N, 40xx:4071N
- added SI4: TSOP-6_PMOS, TSOP-6_MOS:TSOP-6_PMOS
- added U$3: TEENSY40, teensy:TEENSY40
- added U2: SN74HC193QPWRG4Q1, counter_3bit:SN74HC193QPWRG4Q1
- R23: value 1k -> 10k; device IIT_BOMBAY_Racing:R-EU_M0805 -> IIT_BOMBAY_Racing2:R-EU_M0805
Connections:
- net 2V_REF renamed 2VREF
- net 3V3_REF renamed 3V3REF
- net AS_REL_LOGIC renamed AS_RELAY
- net AS_REL_LOGIC_IN renamed AS_RELAY_INV
- net LATCH_OUT_INV renamed AS_LATCH_INV
- net WATCHDOG_OUT renamed WD_OUT
- removed net +12V_AS: C2.2, D1.C, IC5.S_1, IC5.S_2, IC5.S_3, IC7.S_1, IC7.S_2, IC7.S_3, R8.1, R9.1, U$1G$3.V+, U$9.NO+, U$9.V+, X2.9
- removed net ASMS_STATE: IC11A.I1, IC13B.I1, R20.2, SI5.G, U$9.NO-, X2.10
- removed net IN1: IC10A.-IN, IC10A.OUT, IC9.A
- removed net IN1_IN: IC10A.+IN
- removed net IN2: IC10B.-IN, IC10B.OUT, IC9.B
- removed net IN2_IN: IC10B.+IN
- removed net IN3: IC10C.-IN, IC10C.OUT, IC9.C
- removed net IN3_IN: IC10C.+IN
- removed net INIT_CHK_NOT: U1G$1.NON-INVERTING_INPUT1
- removed net INIT_CHK_NOT_12V: IC12C.I1, IC12D.I1, R23.2, U1G$1.OUTPUT1
- removed net LATCH_IN: IC12D.O, IC2.TR
- removed net LATCH_OUT: IC2.Q
- removed net WATCHDOG_OUT_12V: IC11A.I0, U1G$2.OUTPUT2
- new net +12V_ASMS: C11.+, C2.2, D1.C, IC3A.I1, IC4D.I0, IC5.S_1, IC5.S_2, IC5.S_3, IC7.S_1, IC7.S_2, IC7.S_3, R20.2, R8.1, R9.1, SI4.S, SI5.G, U$1G$3.V+, U$9.V+
- new net AMI_0: IC9.A, U2.QA
- new net AMI_1: IC9.B, U2.QB
- new net AMI_2: IC9.C, U2.QC
- new net ASMS_IN: U$9.NO+, X2.9
- new net ASMS_SUPPLY: C10.+, FUSE_1A2.1, U$9.NO-, X2.10
- new net AS_LATCH: IC2.Q, R32.2, SI2.G
- new net AS_TRIG: IC2.TR, IC8D.O
- new net INIT_CHK_INV: IC8B.I0, U1G$1.NON-INVERTING_INPUT1
- new net INIT_CHK_INV_12V: IC8D.I1, K1.DS1, U1G$1.OUTPUT1
- new net N$20: R23.1, U2.CLR, U2.QD
- new net N$21: U2.UP
- new net WD_OUT_12V: IC3A.I0, U1G$2.OUTPUT2
- net +12V: now also IC3P.VDD, IC4P.VDD, IC8P.VDD; no longer IC11P.VDD, IC12P.VDD, IC13P.VDD
- net +5V: now also U2.!LOAD, U2.DOWN, U2.VCC
- net ASMS_STATE_INV: now also IC3D.I0, IC4C.I0; no longer IC13A.I1, IC13C.I0
- net AS_LOGIC: now also IC4B.O, IC8D.I0; no longer IC11D.O, IC12D.I0
- net EBS_RESET: no longer IC2.R, R31.1
- net GND: now also C10.-, C11.-, C12.2, IC3P.VSS, IC4P.VSS, IC8P.VSS, R23.2, SI4.G, U2.A, U2.B, U2.C, U2.D, U2.GND; no longer IC10P.V-, IC11P.VSS, IC12P.VSS, IC13P.VSS
- net HV_RESET: now also IC8A.O; no longer IC12B.O
- net HV_RESET_CP: now also IC4C.I1; no longer IC13A.I0
- net HV_RESET_SP: now also IC8B.I1; no longer IC12C.I0
- net MANUAL_DRIVING: now also IC3D.I1; no longer IC13C.I1, R32.2, SI2.G
- net MANUAL_DRIVING_INV: now also IC3B.I0; no longer IC11B.I0
- net MANUAL_VALVE: now also IC3B.I1; no longer IC11B.I1
- net MANUAL_VALVE_INV: now also IC4A.I1; no longer IC13D.I1
- net MISSION_SET_12V: now also IC4B.I1; no longer IC11D.I1
- net N$10: now also IC3A.O, IC3C.I0; no longer IC11A.O, IC11C.I0
- net N$11: now also IC3B.O, IC3C.I1; no longer IC11B.O, IC11C.I1
- net N$12: now also IC3D.O, IC4A.I0; no longer IC13C.O, IC13D.I0
- net N$17: now also C12.1, IC2.R, R31.1; no longer K1.DS1, R23.1
- net N$2: now also IC4B.I0, IC8C.O; no longer IC11D.I0, IC12A.O
- net N$7: now also FUSE_1A2.2, SI4.1, SI4.2, SI4.5, SI4.6, SI4.D0; no longer IC10P.V+
- net SIG1: now also IC3C.O, IC8C.I0; no longer IC11C.O, IC12A.I0
- net SIG2: now also IC4C.O, IC8A.I0; no longer IC12B.I0, IC13A.O
- net SIG3: now also IC4D.O, IC8A.I1; no longer IC12B.I1, IC13B.O
- net SIG4: now also IC4A.O, IC8C.I1; no longer IC12A.I1, IC13D.O
- net SIG5: now also IC4D.I1, IC8B.O; no longer IC12C.O, IC13B.I0
- net TRACKDRIVE: no longer X2.6
Other:
- note added: "AMI"
- note added: "AS Latch Block"
- note added: "AS Relay Logic"
- note added: "ASSI Block"
- note added: "HV Reset Block"
- note added: "Signal Inversion"
- note added: "Supply voltage cannot be 5V as min input V is .7*VDD"
- note removed: "AS Logic"
- note removed: "ASSI Led Out"
- note removed: "HV Reset"
- note removed: "Supply voltage cannot be 5V as min input V is .7*VDD Input current is 12uA so directly connected +3v3"
